Commit message: update readme and eval on turtlebot data (test*.ods)

File: turtlebot3_description/urdf/turtlebot3_waffle.gazebo.xacro (robot description, xacro)
@@ -133,6 +133,6 @@
           <horizontal_fov>1.3439</horizontal_fov>
           <image>
-              <width>640</width>
-              <height>480</height>
+              <width>320</width>
+              <height>240</height>
               <format>R8G8B8</format>
           </image>

File: turtlebot3_description/urdf/turtlebot3_waffle.urdf.xacro (robot description, xacro)
@@ -91,5 +91,5 @@
       </inertial>
   </link>
-  <joint name="caster_back_right_joint" type="fixed">
+  <joint name="caster_back_right_joint" type="continuous">
     <parent link="base_link"/>
     <child link="caster_back_right_link"/>
@@ -111,5 +111,5 @@
     </inertial>
   </link>
-  <joint name="caster_back_left_joint" type="fixed">
+  <joint name="caster_back_left_joint" type="continuous">
     <parent link="base_link"/>
     <child link="caster_back_left_link"/>
@@ -186,5 +186,5 @@
     <child link="camera_link"/>
         <axis xyz="0 0 1"/>
-    <limit effort="1000.0" lower="0.0" upper="0.548" velocity="0.5"/>
+    <limit effort="1000.0" lower="0.0" upper="0.0" velocity="0.00005"/>
   </joint>
   <link name="camera_link">
@@ -209,10 +209,26 @@
     </inertial>
   </link>
-  <joint name="camera_rgb_joint" type="fixed">
+  <joint name="camera_rgb_joint" type="revolute">
     <origin xyz="${r200_cam_rgb_px} ${r200_cam_rgb_py} ${r200_cam_rgb_pz}" rpy="0 0 0"/>
     <parent link="camera_link"/>
     <child link="camera_rgb_frame"/>
-  </joint>
-  <link name="camera_rgb_frame"/>
+        <axis xyz="0 0 1"/>
+    <limit effort="1000.0" lower="0.0" upper="0.0" velocity="0.0005"/>
+  </joint>
+  <link name="camera_rgb_frame">
+    <collision>
+      <origin xyz="0.0003 0.0003 0.007" rpy="0 0 0"/>
+      <geometry>
+        <box size="0.00012 0.000132 0.00020"/>
+      </geometry>
+    </collision>
+    <inertial>
+      <mass value="0.00114" />
+      <origin xyz="0 0 0" />
+      <inertia ixx="0.001" ixy="0.0" ixz="0.0"
+               iyy="0.001" iyz="0.0"
+               izz="0.001" />
+    </inertial>
+  </link>
   <joint name="camera_rgb_optical_joint" type="fixed">
     <origin xyz="0 0 0" rpy="-1.57 0 -1.57"/>
